File: Hardware/PCB/Modules/IMU.kicad_sch (KiCad schematic)
At the start: 3 parts, among them U5 ICM-20948

Commit message: Update schematic
Parts:
- C? (x2): renamed from C2; footprint Capacitor_SMD:C_0603_1608Metric -> Capacitor_SMD:C_0402_1005Metric
- renumbered U5 to U1
Connections:
- net GND_IMU is gone; now on net GND: C?.2, C?.2, U1.18 (GND), U1.20 (GND)
- net GND: now reaches U1.12 (INT1)
- net IMU_SCL renamed I2C_LevelShifter/SCL_LL
- net IMU_SDA renamed I2C_LevelShifter/SDA_LL
- net VCC_IN renamed +3.3V
- no-connect marks 0 -> 4
Other:
- added sheet I2C_LevelShifter (LevelShifter.kicad_sch)

Commit message: Update of PCB and schematic
Parts:
- removed U1: ICM-20948, Sensor_Motion:InvenSense_QFN-24_3x3mm_P0.4mm, symbol Sensor_Motion:ICM-20948
- added C?: 100nF, Capacitor_SMD:C_0603_1608Metric, symbol Device:C
- added R3: 47k, Resistor_SMD:R_0603_1608Metric, symbol Device:R
- added U8: MPU-9250, Sensor_Motion:InvenSense_QFN-24_3x3mm_P0.4mm, symbol Sensor_Motion:MPU-9250
- C? (x2): footprint Capacitor_SMD:C_0402_1005Metric -> Capacitor_SMD:C_0603_1608Metric
Connections:
- net +3.3V: now also U8.1 (RESV_VDDIO), U8.13 (VDD), U8.22 (~{CS}), U8.8 (VDDIO)
- net GND: now also C?.2, R3.2, U8.18 (GND), U8.20 (RESV_GND)
- net SCL: now also U8.23 (SCL/SCLK)
- net SDA: now also U8.24 (SDA/MOSI)
- new net: R3.1, U8.11 (FSYNC)
- new net: C?.1, U8.10 (REGOUT)
- no-connect marks 4 -> 7
Other:
- removed sheet I2C_LevelShifter

Commit message: update of directory
Parts:
- gave numbers to parts that had none: 3
- renumbered R3 to R19
