File: Hardware/PCB/Modules/EEPROM.kicad_sch (KiCad schematic)
At the start: 7 parts, among them U5 MPU-9250

Commit message: save
Parts:
- removed C10, C16, C8: 100nF, Capacitor_SMD:C_0603_1608Metric, symbol Device:C
- removed R23, R24, R25: 10k, Resistor_SMD:R_0603_1608Metric, symbol Device:R
- removed U5: MPU-9250, Sensor_Motion:InvenSense_QFN-24_3x3mm_P0.4mm, symbol Sensor_Motion:MPU-9250
- added C17: 100nF, Capacitor_SMD:C_0603_1608Metric, symbol Device:C
- added R27, R28, R29, R30, R31, R32, R33: 10k, Resistor_SMD:R_0603_1608Metric, symbol Device:R
- added U9: 24LC64, Package_SO:SOIC-8-1EP_3.9x4.9mm_P1.27mm_EP2.29x3mm, symbol Memory_EEPROM:24LC64
Connections:
- net +3.3V: now also C17.2, R31.1, R32.1, R33.1, U9.8 (VCC)
- net GND: now also C17.1, R27.2, R28.2, R29.2, R30.2, U9.4 (GND)
- net SCL: now also U9.6 (SCL)
- net SDA: now also U9.5 (SDA)
- new net: R30.1, R33.2, U9.1 (A0)
- new net: R29.1, R32.2, U9.2 (A1)
- new net: R28.1, R31.2, U9.3 (A2)
- new net: R27.1, U9.7 (WP)
- no-connect marks 4 -> 0
