File: Hardware/PCB/Modules/Key.kicad_sch (KiCad schematic)
At the start: 3 parts, among them SW1 SW_HotSwap

Commit message: Update of schematic and PCB
Other:
- moved on the sheet: D13
Changed lines of the file:
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@@
   (junction (at 60.96 72.39) (diameter 0) (color 0 0 0 0)
   )
-  (wire (pts (xy 135.89 60.96) (xy 138.43 60.96))
+  (wire (pts (xy 118.11 62.23) (xy 120.65 62.23))
     (stroke (width 0) (type default))
   )
-  (wire (pts (xy 146.05 68.58) (xy 146.05 76.2))
+  (wire (pts (xy 128.27 69.85) (xy 128.27 77.47))
     (stroke (width 0) (type default))
   )
@@
     (stroke (width 0) (type default))
   )
-  (wire (pts (xy 153.67 60.96) (xy 156.21 60.96))
+  (wire (pts (xy 135.89 62.23) (xy 138.43 62.23))
     (stroke (width 0) (type default))
   )
@@
     (stroke (width 0) (type default))
   )
-  (wire (pts (xy 146.05 41.91) (xy 146.05 53.34))
+  (wire (pts (xy 128.27 43.18) (xy 128.27 54.61))
     (stroke (width 0) (type default))
   )
@@
     (stroke (width 0) (type default))
   )
-  (hierarchical_label "Led_Input" (shape input) (at 135.89 60.96 180) (fields_autoplaced)
+  (hierarchical_label "Led_Input" (shape input) (at 118.11 62.23 180) (fields_autoplaced)
     (effects (font (size 1.27 1.27)) (justify right))
   )
-  (hierarchical_label "Vdd" (shape input) (at 146.05 41.91 90) (fields_autoplaced)
+  (hierarchical_label "Vdd" (shape input) (at 128.27 43.18 90) (fields_autoplaced)
     (effects (font (size 1.27 1.27)) (justify left))
   )
@@
     (effects (font (size 1.27 1.27)) (justify right))
   )
-  (hierarchical_label "GND" (shape output) (at 146.05 76.2 270) (fields_autoplaced)
+  (hierarchical_label "GND" (shape output) (at 128.27 77.47 270) (fields_autoplaced)
     (effects (font (size 1.27 1.27)) (justify right))
   )
@@
     (effects (font (size 1.27 1.27)) (justify right))
   )
-  (hierarchical_label "Led_Output" (shape output) (at 156.21 60.96 0) (fields_autoplaced)
+  (hierarchical_label "Led_Output" (shape output) (at 138.43 62.23 0) (fields_autoplaced)
     (effects (font (size 1.27 1.27)) (justify left))
   )
@@
     )
   )
-  (symbol (lib_id "LED:SK6812MINI") (at 146.05 60.96 0) (unit 1)
+  (symbol (lib_id "LED:SK6812MINI") (at 128.27 62.23 0) (unit 1)
     (in_bom yes) (on_board yes) (dnp no)
-    (property "Reference" "D13" (at 149.86 54.61 0)
+    (property "Reference" "D13" (at 132.08 55.88 0)
       (effects (font (size 1.27 1.27)))
     )
-    (property "Value" "SK6812MINI" (at 158.75 60.3759 0)
+    (property "Value" "SK6812MINI" (at 140.97 61.6459 0)
       (effects (font (size 1.27 1.27)) hide)
     )
-    (property "Footprint" "LED_SMD:LED_SK6812MINI_PLCC4_3.5x3.5mm_P1.75mm" (at 147.32 68.58 0)
+    (property "Footprint" "LED_SMD:LED_SK6812MINI_PLCC4_3.5x3.5mm_P1.75mm" (at 129.54 69.85 0)
       (effects (font (size 1.27 1.27)) (justify left top) hide)
     )
-    (property "Datasheet" "https://cdn-shop.adafruit.com/product-files/2686/SK6812MINI_REV.01-1-2.pdf" (at 148.59 70.485 0)
+    (property "Datasheet" "https://cdn-shop.adafruit.com/product-files/2686/SK6812MINI_REV.01-1-2.pdf" (at 130.81 71.755 0)
       (effects (font (size 1.27 1.27)) (justify left top) hide)
     )

Commit message: update of directory
Parts:
- D2: renamed from D13; value SK6812MINI -> SK6812MINI-E

Commit message: save
Parts:
- renumbered D2 to D1, D1 to D11
Changed lines of the file:
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@@
 		(dnp no)
 		(fields_autoplaced yes)
-		(property "Reference" "D1"
+		(property "Reference" "D11"
 			(at 63.5 61.595 90)
 			(effects
@@
 			(project "PCB"
 				(path "/fd8c8265-4947-4b90-b980-57cac1b7867b/416eee54-53c7-4fdf-9784-49e18a35f298"
-					(reference "D1")
+					(reference "D11")
 					(unit 1)
 				)
@@
 		(on_board yes)
 		(dnp no)
-		(property "Reference" "D2"
+		(property "Reference" "D1"
 			(at 132.08 55.88 0)
 			(effects
@@
 			(project "PCB"
 				(path "/fd8c8265-4947-4b90-b980-57cac1b7867b/416eee54-53c7-4fdf-9784-49e18a35f298"
-					(reference "D2")
+					(reference "D1")
 					(unit 1)
 				)
