File: Hardware/PCB/Modules/LevelShifter.kicad_sch (KiCad schematic)
At the start: 6 parts, among them Q3 PJC138K_R1_00001

Commit message: update of directory
Parts:
- R20, R21, R22, R23: renamed from R?; footprint Resistor_SMD:R_0402_1005Metric -> Resistor_SMD:R_0603_1608Metric
- renumbered Q3 to Q4

Commit message: save
Parts:
- renumbered Q4 to Q3, Q3 to Q4, R23 to R17, R20 to R18, R21 to R19, R22 to R21
Changed lines of the file:
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@@
 		(on_board yes)
 		(dnp no)
-		(property "Reference" "R21"
+		(property "Reference" "R19"
 			(at 137.16 68.58 0)
 			(effects
@@
 			(project "PCB"
 				(path "/fd8c8265-4947-4b90-b980-57cac1b7867b/fd9ec7b9-711c-46f0-80ac-a30badd88661/10818d9a-65b8-46a4-bb9c-7776114cc710"
-					(reference "R21")
+					(reference "R19")
 					(unit 1)
 				)
@@
 		(dnp no)
 		(fields_autoplaced yes)
-		(property "Reference" "Q4"
+		(property "Reference" "Q3"
 			(at 143.51 102.87 90)
 			(effects
@@
 			(project "PCB"
 				(path "/fd8c8265-4947-4b90-b980-57cac1b7867b/fd9ec7b9-711c-46f0-80ac-a30badd88661/10818d9a-65b8-46a4-bb9c-7776114cc710"
-					(reference "Q4")
+					(reference "Q3")
 					(unit 1)
 				)
@@
 		(on_board yes)
 		(dnp no)
-		(property "Reference" "R23"
+		(property "Reference" "R17"
 			(at 152.4 68.58 0)
 			(effects
@@
 			(project "PCB"
 				(path "/fd8c8265-4947-4b90-b980-57cac1b7867b/fd9ec7b9-711c-46f0-80ac-a30badd88661/10818d9a-65b8-46a4-bb9c-7776114cc710"
-					(reference "R23")
+					(reference "R17")
 					(unit 1)
 				)
@@
 		(on_board yes)
 		(dnp no)
-		(property "Reference" "R20"
+		(property "Reference" "R18"
 			(at 135.89 91.44 0)
 			(effects
@@
 			(project "PCB"
 				(path "/fd8c8265-4947-4b90-b980-57cac1b7867b/fd9ec7b9-711c-46f0-80ac-a30badd88661/10818d9a-65b8-46a4-bb9c-7776114cc710"
-					(reference "R20")
+					(reference "R18")
 					(unit 1)
 				)
@@
 		(on_board yes)
 		(dnp no)
-		(property "Reference" "Q3"
+		(property "Reference" "Q4"
 			(at 144.78 80.01 90)
 			(effects
@@
 			(project "PCB"
 				(path "/fd8c8265-4947-4b90-b980-57cac1b7867b/fd9ec7b9-711c-46f0-80ac-a30badd88661/10818d9a-65b8-46a4-bb9c-7776114cc710"
-					(reference "Q3")
+					(reference "Q4")
 					(unit 1)
 				)
@@
 		(on_board yes)
 		(dnp no)
-		(property "Reference" "R22"
+		(property "Reference" "R21"
 			(at 151.13 91.44 0)
 			(effects
@@
 			(project "PCB"
 				(path "/fd8c8265-4947-4b90-b980-57cac1b7867b/fd9ec7b9-711c-46f0-80ac-a30badd88661/10818d9a-65b8-46a4-bb9c-7776114cc710"
-					(reference "R22")
-					(unit 1)
-				)
+					(reference "R21")
+					(unit 1)
+				)
