File: Hardware/PCB/Modules/MCU.kicad_sch.kicad_sch (KiCad schematic)
At the start: 11 parts, among them U3 STM32F303RETx, X1 ECS-2520MV-250-DN-TR

Commit message: Update schematic
Parts:
- added R15, R16: 0, Resistor_SMD:R_0402_1005Metric, symbol Device:R
- C5, C7, C8: footprint Capacitor_SMD:C_0603_1608Metric -> Capacitor_SMD:C_0402_1005Metric
- R5, R6: footprint Resistor_SMD:R_0603_1608Metric -> Resistor_SMD:R_0402_1005Metric
- R7: renamed from R10; footprint Resistor_SMD:R_0603_1608Metric -> Resistor_SMD:R_0402_1005Metric
- R7: renamed from R11; footprint Resistor_SMD:R_0603_1608Metric -> Resistor_SMD:R_0402_1005Metric
Connections:
- net SCL_MCU is gone; now on net SCL: R7.2
- net SDA_MCU is gone; now on net SDA: R7.2
- net at U3.46 (PA13): now also R15.1
- net at U3.49 (PA14): now also R16.1
- net SDA: now reaches U3.57 (PB5)
- net SCL: now reaches U3.58 (PB6)
- net GND_MCU renamed GND
- net VCC_IN renamed +3.3V
- new net SWC: R16.2
- new net SWD: R15.2
Other:
- moved on the sheet: R7

Commit message: Update of PCB and schematic
Parts:
- added R7: 220, Resistor_SMD:R_0402_1005Metric, symbol Device:R
- C5, C7, C8: footprint Capacitor_SMD:C_0402_1005Metric -> Capacitor_SMD:C_0603_1608Metric
Connections:
- net GND: now also U3.60 (BOOT0)
- net TX: now reaches U3.42 (PA9)
- net RX: now reaches U3.43 (PA10)
- net at U3.62 (PB9): now also R7.1
- new net IR_LED: R7.2
Changed lines of the file:
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@@
+    (stroke (width 0) (type default))
+  )
+  (wire (pts (xy 154.94 90.17) (xy 171.45 90.17))
     (stroke (width 0) (type default))
   )
@@
     (stroke (width 0) (type default))
   )
+  (wire (pts (xy 154.94 87.63) (xy 171.45 87.63))
+    (stroke (width 0) (type default))
+  )
   (wire (pts (xy 77.47 87.63) (xy 77.47 90.17))
     (stroke (width 0) (type default))
@@
     (stroke (width 0) (type default))
   )
+  (wire (pts (xy 113.03 69.85) (xy 119.38 69.85))
+    (stroke (width 0) (type default))
+  )
   (bus (pts (xy 176.53 116.84) (xy 184.15 116.84))
     (stroke (width 0) (type default))
@@
   )
   (wire (pts (xy 167.64 100.33) (xy 171.45 100.33))
+    (stroke (width 0) (type default))
+  )
+  (wire (pts (xy 154.94 130.81) (xy 156.21 130.81))
     (stroke (width 0) (type default))
   )
@@
     (effects (font (size 1.27 1.27)) (justify left bottom))
   )
+  (label "IR_LED" (at 163.83 130.81 0) (fields_autoplaced)
+    (effects (font (size 1.27 1.27)) (justify left bottom))
+  )
   (hierarchical_label "USB-" (shape bidirectional) (at 171.45 95.25 0) (fields_autoplaced)
     (effects (font (size 1.27 1.27)) (justify left))
@@
     (effects (font (size 1.27 1.27)) (justify left))
   )
+  (hierarchical_label "TX" (shape output) (at 171.45 87.63 0) (fields_autoplaced)
+    (effects (font (size 1.27 1.27)) (justify left))
+  )
+  (hierarchical_label "GND" (shape passive) (at 113.03 69.85 180) (fields_autoplaced)
+    (effects (font (size 1.27 1.27)) (justify right))
+  )
   (hierarchical_label "GND" (shape output) (at 116.84 55.88 270) (fields_autoplaced)
     (effects (font (size 1.27 1.27)) (justify right))
@@
     (effects (font (size 1.27 1.27)) (justify right))
   )
-  (hierarchical_label "GND" (shape output) (at 92.71 93.98 270) (fields_autoplaced)
-    (effects (font (size 1.27 1.27)) (justify right))
-  )
-  (hierarchical_label "GND" (shape output) (at 138.43 167.64 270) (fields_autoplaced)
+  (hierarchical_label "GND" (shape passive) (at 92.71 93.98 270) (fields_autoplaced)
+    (effects (font (size 1.27 1.27)) (justify right))
+  )
+  (hierarchical_label "RX" (shape input) (at 171.45 90.17 0) (fields_autoplaced)
+    (effects (font (size 1.27 1.27)) (justify left))
+  )
+  (hierarchical_label "GND" (shape passive) (at 138.43 167.64 270) (fields_autoplaced)
     (effects (font (size 1.27 1.27)) (justify right))
   )
@@
       (effects (font (size 1.27 1.27)) (justify left))
     )
-    (property "Footprint" "Capacitor_SMD:C_0402_1005Metric" (at 152.0952 55.88 0)
+    (property "Footprint" "Capacitor_SMD:C_0603_1608Metric" (at 152.0952 55.88 0)
       (effects (font (size 1.27 1.27)) hide)
     )
@@
     )
   )
+  (symbol (lib_id "Device:R") (at 160.02 130.81 90) (mirror x) (unit 1)
+    (in_bom yes) (on_board yes) (dnp no)
+    (property "Reference" "R7" (at 160.02 128.27 90)
+      (effects (font (size 1.27 1.27)))
+    )
+    (property "Value" "220" (at 160.02 130.81 90)
+      (effects (font (size 1.27 1.27)))
+    )
+    (property "Footprint" "Resistor_SMD:R_0402_1005Metric" (at 160.02 129.032 90)
+      (effects (font (size 1.27 1.27)) hide)
+    )
+    (property "Datasheet" "~" (at 160.02 130.81 0)
+      (effects (font (size 1.27 1.27)) hide)
+    )
+    (pin "1")
+    (pin "2")
+    (instances
+      (project "PCB"
+        (path "/fd8c8265-4947-4b90-b980-57cac1b7867b/ac97498d-2051-444b-8e34-d771fa4cf1f1"
+          (reference "R7") (unit 1)
+        )
+        (path "/fd8c8265-4947-4b90-b980-57cac1b7867b/21016d7c-fd8b-4404-8ef7-6ca90f156ddd"
+          (reference "R9") (unit 1)
+        )
+        (path "/fd8c8265-4947-4b90-b980-57cac1b7867b/5826a8b9-a512-49e5-9762-3dc7f408520c"
+          (reference "R18") (unit 1)
+        )
+      )
+    )
+  )
   (symbol (lib_id "Device:C") (at 116.84 52.07 0) (unit 1)
     (in_bom yes) (on_board yes) (dnp no)
@@
       (effects (font (size 1.27 1.27)) (justify left))
     )
-    (property "Footprint" "Capacitor_SMD:C_0402_1005Metric" (at 117.8052 55.88 0)
+    (property "Footprint" "Capacitor_SMD:C_0603_1608Metric" (at 117.8052 55.88 0)
       (effects (font (size 1.27 1.27)) hide)
     )
@@
       (effects (font (size 1.27 1.27)) (justify left))
     )
-    (property "Footprint" "Capacitor_SMD:C_0402_1005Metric" (at 78.4352 87.63 0)
+    (property "Footprint" "Capacitor_SMD:C_0603_1608Metric" (at 78.4352 87.63 0)
       (effects (font (size 1.27 1.27)) hide)
     )
@@
       (effects (font (size 1.27 1.27)) (justify left))
     )
-    (property "Footprint" "Capacitor_SMD:C_0402_1005Metric" (at 163.5252 55.88 0)
-      (effects (font (size 1.27 1.27)) hide)
-    )
+    (property "Footprint" "Capacitor_SMD:C_0603_1608Metric" (at 163.5252 55.88 0)
+      (effects (font (size 1.27 1.27)) hide)
+    )

Commit message: update of directory
Parts:
- R10, R11, R18: renamed from R7; footprint Resistor_SMD:R_0402_1005Metric -> Resistor_SMD:R_0603_1608Metric
- R15, R16, R5, R6: footprint Resistor_SMD:R_0402_1005Metric -> Resistor_SMD:R_0603_1608Metric
- renumbered C8 to C13, C8 to C5, C5 to C7, C7 to C8

Commit message: save
Parts:
- removed C6: 470nF, Capacitor_SMD:C_0603_1608Metric, symbol Device:C
- added C1, C2, C7: 100nF, Capacitor_SMD:C_0603_1608Metric, symbol Device:C
- added R26: 10, Resistor_SMD:R_0603_1608Metric, symbol Device:R
- added R6: 0, Resistor_SMD:R_0603_1608Metric, symbol Device:R
- renumbered C8 to C11, C7 to C13, C13 to C15, C5 to C3, R16 to R10, R5 to R13, R6 to R14, R18 to R20, R10 to R22, U3 to U2
Connections:
- net +3.3V: now also C1.1, C2.1, C7.1
- net GND: now also C1.2, C2.2, C7.2, R6.1; no longer U2.60 (BOOT0)
- net at U2.5 (PF0): now also R26.2; no longer X1.3 (OUT)
- new net: R6.2, U2.60 (BOOT0)
- new net: R26.1, X1.3 (OUT)
Other:
- moved on the sheet: C11
