File: Hardware/PCB/Modules/Multimeter.kicad_sch (KiCad schematic)
At the start: 10 parts, among them Q2 NMOS, U4 MC1413BD

Commit message: Update of PCB and schematic
Changed lines of the file:
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@@
   (junction (at 140.97 81.28) (diameter 0) (color 0 0 0 0)
-  )
-  (junction (at 119.38 44.45) (diameter 0) (color 0 0 0 0)
   )
   (junction (at 102.87 107.95) (diameter 0) (color 0 0 0 0)
@@
     (stroke (width 0) (type default))
   )
-  (wire (pts (xy 115.57 44.45) (xy 119.38 44.45))
-    (stroke (width 0) (type default))
-  )
   (wire (pts (xy 125.73 102.87) (xy 148.59 102.87))
     (stroke (width 0) (type default))
@@
     (stroke (width 0) (type default))
   )
-  (wire (pts (xy 115.57 49.53) (xy 119.38 49.53))
-    (stroke (width 0) (type default))
-  )
   (wire (pts (xy 102.87 110.49) (xy 105.41 110.49))
     (stroke (width 0) (type default))
@@
     (stroke (width 0) (type default))
   )
-  (wire (pts (xy 119.38 49.53) (xy 119.38 44.45))
-    (stroke (width 0) (type default))
-  )
   (wire (pts (xy 148.59 102.87) (xy 148.59 93.98))
     (stroke (width 0) (type default))
@@
     (stroke (width 0) (type default))
   )
-  (wire (pts (xy 119.38 44.45) (xy 124.46 44.45))
+  (wire (pts (xy 115.57 44.45) (xy 124.46 44.45))
     (stroke (width 0) (type default))
   )
@@
     (effects (font (size 1.27 1.27)) (justify left bottom))
   )
+  (hierarchical_label "+5V" (shape input) (at 115.57 44.45 180) (fields_autoplaced)
+    (effects (font (size 1.27 1.27)) (justify right))
+  )
   (hierarchical_label "GND" (shape output) (at 115.57 128.27 270) (fields_autoplaced)
     (effects (font (size 1.27 1.27)) (justify right))
   )
-  (hierarchical_label "VCC_IN" (shape input) (at 115.57 44.45 180) (fields_autoplaced)
-    (effects (font (size 1.27 1.27)) (justify right))
-  )
-  (hierarchical_label "VCC_OUT" (shape output) (at 115.57 49.53 180) (fields_autoplaced)
-    (effects (font (size 1.27 1.27)) (justify right))
-  )

Commit message: update of directory
Parts:
- R12, R13, R7, R8, R9: renamed from R?; footprint Resistor_SMD:R_0805_2012Metric -> Resistor_SMD:R_0603_1608Metric
- gave numbers to parts that had none: 1
- renumbered R4 to R14

Commit message: save
Parts:
- renumbered D7 to D3, D6 to D4, Q2 to Q1, R8 to R1, R9 to R2, R7 to R4, R13 to R7, R14 to R8, R12 to R9, U4 to U3
Changed lines of the file:
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@@
 		(dnp no)
 		(fields_autoplaced yes)
-		(property "Reference" "R7"
+		(property "Reference" "R4"
 			(at 143.51 68.58 0)
 			(effects
@@
 			(project "PCB"
 				(path "/fd8c8265-4947-4b90-b980-57cac1b7867b/c429b47e-7556-484b-b844-f8d6007e758d"
-					(reference "R7")
+					(reference "R4")
 					(unit 1)
 				)
@@
 		(on_board yes)
 		(dnp no)
-		(property "Reference" "R13"
+		(property "Reference" "R7"
 			(at 144.78 86.36 0)
 			(effects
@@
 			(project "PCB"
 				(path "/fd8c8265-4947-4b90-b980-57cac1b7867b/c429b47e-7556-484b-b844-f8d6007e758d"
-					(reference "R13")
+					(reference "R7")
 					(unit 1)
 				)
@@
 		(dnp no)
 		(fields_autoplaced yes)
-		(property "Reference" "R14"
+		(property "Reference" "R8"
 			(at 114.3 75.565 0)
 			(effects
@@
 			(project "PCB"
 				(path "/fd8c8265-4947-4b90-b980-57cac1b7867b/c429b47e-7556-484b-b844-f8d6007e758d"
-					(reference "R14")
+					(reference "R8")
 					(unit 1)
 				)
@@
 		(on_board yes)
 		(dnp no)
-		(property "Reference" "R9"
+		(property "Reference" "R2"
 			(at 129.54 86.36 0)
 			(effects
@@
 			(project "PCB"
 				(path "/fd8c8265-4947-4b90-b980-57cac1b7867b/c429b47e-7556-484b-b844-f8d6007e758d"
-					(reference "R9")
+					(reference "R2")
 					(unit 1)
 				)
@@
 		(on_board yes)
 		(dnp no)
-		(property "Reference" "R12"
+		(property "Reference" "R9"
 			(at 139.7 86.36 0)
 			(effects
@@
 			(project "PCB"
 				(path "/fd8c8265-4947-4b90-b980-57cac1b7867b/c429b47e-7556-484b-b844-f8d6007e758d"
-					(reference "R12")
+					(reference "R9")
 					(unit 1)
 				)
@@
 		(on_board yes)
 		(dnp no)
-		(property "Reference" "Q2"
+		(property "Reference" "Q1"
 			(at 119.38 66.04 0)
 			(effects
@@
 			(project "PCB"
 				(path "/fd8c8265-4947-4b90-b980-57cac1b7867b/c429b47e-7556-484b-b844-f8d6007e758d"
-					(reference "Q2")
+					(reference "Q1")
 					(unit 1)
 				)
@@
 		(on_board yes)
 		(dnp no)
-		(property "Reference" "R8"
+		(property "Reference" "R1"
 			(at 134.62 86.36 0)
 			(effects
@@
 			(project "PCB"
 				(path "/fd8c8265-4947-4b90-b980-57cac1b7867b/c429b47e-7556-484b-b844-f8d6007e758d"
-					(reference "R8")
+					(reference "R1")
 					(unit 1)
 				)
@@
 		(on_board yes)
 		(dnp no)
-		(property "Reference" "D6"
+		(property "Reference" "D4"
 			(at 124.46 74.93 0)
 			(effects
@@
 			(project "PCB"
 				(path "/fd8c8265-4947-4b90-b980-57cac1b7867b/c429b47e-7556-484b-b844-f8d6007e758d"
-					(reference "D6")
+					(reference "D4")
 					(unit 1)
 				)
@@
 		(dnp no)
 		(fields_autoplaced yes)
-		(property "Reference" "D7"
+		(property "Reference" "D3"
 			(at 160.02 88.9 90)
 			(effects
@@
 			(project "PCB"
 				(path "/fd8c8265-4947-4b90-b980-57cac1b7867b/c429b47e-7556-484b-b844-f8d6007e758d"
-					(reference "D7")
+					(reference "D3")
 					(unit 1)
 				)
@@
 		(on_board yes)
 		(dnp no)
-		(property "Reference" "U4"
+		(property "Reference" "U3"
 			(at 115.57 82.55 0)
 			(effects
@@
 			(project "PCB"
 				(path "/fd8c8265-4947-4b90-b980-57cac1b7867b/c429b47e-7556-484b-b844-f8d6007e758d"
-					(reference "U4")
-					(unit 1)
-				)
+					(reference "U3")
+					(unit 1)
+				)
