File: Hardware/PCB/Modules/OLED.kicad_sch (KiCad schematic)
At the start: 1 part, among them J3 I2C_SSD1306

Commit message: Update of PCB and schematic
Connections:
- net SCL: no longer J3.2 (Pin_2)
- net SDA: no longer J3.3 (Pin_3)
- net VCC_IN renamed +5V
- new net LevelShifter/SCL_HL: J3.2 (Pin_2)
- new net LevelShifter/SDA_HL: J3.3 (Pin_3)
Other:
- added sheet LevelShifter (LevelShifter.kicad_sch)
Changed lines of the file:
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@@
 (kicad_sch (version 20230121) (generator eeschema)
   (paper "A4")
-  (junction (at 156.21 66.04) (diameter 0) (color 0 0 0 0)
+  (junction (at 151.13 66.04) (diameter 0) (color 0 0 0 0)
   )
-  (bus_entry (at 137.16 82.55) (size -2.54 -2.54)
+  (bus_entry (at 110.49 82.55) (size -2.54 -2.54)
     (stroke (width 0) (type default))
   )
-  (bus_entry (at 139.7 82.55) (size -2.54 -2.54)
+  (bus_entry (at 113.03 82.55) (size -2.54 -2.54)
     (stroke (width 0) (type default))
   )
@@
     (stroke (width 0) (type default))
   )
-  (wire (pts (xy 139.7 83.82) (xy 153.67 83.82))
+  (bus (pts (xy 107.95 80.01) (xy 100.33 80.01))
     (stroke (width 0) (type default))
   )
-  (bus (pts (xy 134.62 80.01) (xy 127 80.01))
+  (wire (pts (xy 130.81 66.04) (xy 135.89 66.04))
     (stroke (width 0) (type default))
   )
-  (wire (pts (xy 139.7 82.55) (xy 139.7 83.82))
+  (wire (pts (xy 113.03 82.55) (xy 113.03 83.82))
     (stroke (width 0) (type default))
   )
-  (wire (pts (xy 137.16 86.36) (xy 153.67 86.36))
+  (wire (pts (xy 135.89 66.04) (xy 135.89 80.01))
     (stroke (width 0) (type default))
   )
-  (wire (pts (xy 160.02 66.04) (xy 156.21 66.04))
+  (wire (pts (xy 110.49 86.36) (xy 124.46 86.36))
     (stroke (width 0) (type default))
   )
-  (wire (pts (xy 137.16 82.55) (xy 137.16 86.36))
+  (wire (pts (xy 149.86 86.36) (xy 153.67 86.36))
+    (stroke (width 0) (type default))
+  )
+  (wire (pts (xy 149.86 83.82) (xy 153.67 83.82))
+    (stroke (width 0) (type default))
+  )
+  (wire (pts (xy 113.03 83.82) (xy 124.46 83.82))
+    (stroke (width 0) (type default))
+  )
+  (wire (pts (xy 110.49 82.55) (xy 110.49 86.36))
     (stroke (width 0) (type default))
   )
@@
     (stroke (width 0) (type default))
   )
-  (wire (pts (xy 160.02 60.96) (xy 156.21 60.96))
-    (stroke (width 0) (type default))
-  )
   (wire (pts (xy 151.13 66.04) (xy 151.13 81.28))
     (stroke (width 0) (type default))
   )
-  (bus (pts (xy 137.16 80.01) (xy 134.62 80.01))
+  (bus (pts (xy 110.49 80.01) (xy 107.95 80.01))
     (stroke (width 0) (type default))
   )
-  (wire (pts (xy 156.21 60.96) (xy 156.21 66.04))
+  (wire (pts (xy 138.43 80.01) (xy 138.43 66.04))
     (stroke (width 0) (type default))
   )
-  (wire (pts (xy 156.21 66.04) (xy 151.13 66.04))
+  (wire (pts (xy 151.13 66.04) (xy 160.02 66.04))
+    (stroke (width 0) (type default))
+  )
+  (wire (pts (xy 138.43 66.04) (xy 151.13 66.04))
     (stroke (width 0) (type default))
   )
@@
     (stroke (width 0) (type default))
   )
-  (label "SCL" (at 144.78 86.36 0) (fields_autoplaced)
+  (label "SCL" (at 118.11 86.36 0) (fields_autoplaced)
     (effects (font (size 1.27 1.27)) (justify left bottom))
   )
-  (label "SDA" (at 144.78 83.82 0) (fields_autoplaced)
+  (label "SDA" (at 118.11 83.82 0) (fields_autoplaced)
     (effects (font (size 1.27 1.27)) (justify left bottom))
+  )
+  (hierarchical_label "+3.3V" (shape input) (at 130.81 66.04 180) (fields_autoplaced)
+    (effects (font (size 1.27 1.27)) (justify right))
+  )
+  (hierarchical_label "{SDA SCL}" (shape bidirectional) (at 100.33 80.01 180) (fields_autoplaced)
+    (effects (font (size 1.27 1.27)) (justify right))
+  )
+  (hierarchical_label "+5V" (shape input) (at 160.02 66.04 0) (fields_autoplaced)
+    (effects (font (size 1.27 1.27)) (justify left))
   )
   (hierarchical_label "GND" (shape output) (at 151.13 99.06 270) (fields_autoplaced)
     (effects (font (size 1.27 1.27)) (justify right))
-  )
-  (hierarchical_label "{SDA SCL}" (shape bidirectional) (at 127 80.01 180) (fields_autoplaced)
-    (effects (font (size 1.27 1.27)) (justify right))
-  )
-  (hierarchical_label "VCC_IN" (shape input) (at 160.02 66.04 0) (fields_autoplaced)
-    (effects (font (size 1.27 1.27)) (justify left))
-  )
-  (hierarchical_label "VCC_OUT" (shape output) (at 160.02 60.96 0) (fields_autoplaced)
-    (effects (font (size 1.27 1.27)) (justify left))
   )
   (symbol (lib_id "Connector:Conn_01x04_Pin") (at 158.75 86.36 180) (unit 1)
@@
       )
     )
+  )
+  (sheet (at 124.46 80.01) (size 25.4 8.89) (fields_autoplaced)
+    (stroke (width 0.1524) (type solid))
+    (fill (color 0 0 0 0.0000))
+    (property "Sheetname" "LevelShifter" (at 124.46 79.2984 0)
+      (effects (font (size 1.27 1.27)) (justify left bottom))
+    )
+    (property "Sheetfile" "LevelShifter.kicad_sch" (at 124.46 89.4846 0)
+      (effects (font (size 1.27 1.27)) (justify left top) hide)
+    )
+    (pin "SCL_HL" bidirectional (at 149.86 86.36 0)
+      (effects (font (size 1.27 1.27)) (justify right))
+    )
+    (pin "SDA_HL" bidirectional (at 149.86 83.82 0)
+      (effects (font (size 1.27 1.27)) (justify right))
+    )
+    (pin "SCL_LL" bidirectional (at 124.46 86.36 180)
+      (effects (font (size 1.27 1.27)) (justify left))
+    )
+    (pin "VCC_HL" input (at 138.43 80.01 90)
+      (effects (font (size 1.27 1.27)) (justify right))
+    )
+    (pin "VCC_LL" input (at 135.89 80.01 90)
+      (effects (font (size 1.27 1.27)) (justify right))
+    )
+    (pin "SDA_LL" bidirectional (at 124.46 83.82 180)
+      (effects (font (size 1.27 1.27)) (justify left))
+    )
+    (instances
+      (project "PCB"
+        (path "/fd8c8265-4947-4b90-b980-57cac1b7867b/fd9ec7b9-711c-46f0-80ac-a30badd88661" (page "13"))
+      )
+    )

Commit message: update of directory
Parts:
- renumbered J3 to J2

Commit message: save
Parts:
- added C19, C20: 1µF, Capacitor_SMD:C_0603_1608Metric, symbol Device:C
- added DS1: OLED-128O064D, Display:OLED-128O064D, symbol Display_Graphic:OLED-128O064D
- renumbered J2 to J5
Connections:
- new net: DS1.1 (GND), DS1.30 (GND)
