File: Hardware/PCB/Modules/Programming_sch.kicad_sch (KiCad schematic)
At the start: 6 parts, among them Q1 NMOS

Commit message: Update of schematic and PCB
Parts:
- added C4: 100nF, Capacitor_SMD:C_0603_1608Metric, symbol Device:C
- C4: footprint Capacitor_SMD:C_0805_2012Metric -> Capacitor_SMD:C_0603_1608Metric
- D5: footprint LED_SMD:LED-APA102-2020 -> LED_SMD:LED_0805_2012Metric
- D7: value 1N4818 -> BAS16HT1G; footprint Capacitor_SMD:C_0805_2012Metric -> Diode_SMD:D_SOD-323
- Q1: footprint (none) -> Package_TO_SOT_SMD:SOT-23
Connections:
- net +5V_IN: now also C4.1
- net GND: now also C4.2
Other:
- moved on the sheet: C4
Changed lines of the file:
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@@
     (rev "1")
   )
-  (junction (at 96.52 41.91) (diameter 0) (color 0 0 0 0)
+  (junction (at 82.55 91.44) (diameter 0) (color 0 0 0 0)
+  )
+  (junction (at 76.2 91.44) (diameter 0) (color 0 0 0 0)
   )
   (junction (at 82.55 81.28) (diameter 0) (color 0 0 0 0)
   )
+  (junction (at 76.2 41.91) (diameter 0) (color 0 0 0 0)
+  )
   (junction (at 82.55 52.07) (diameter 0) (color 0 0 0 0)
   )
   (junction (at 92.71 91.44) (diameter 0) (color 0 0 0 0)
   )
+  (junction (at 67.31 55.88) (diameter 0) (color 0 0 0 0)
+  )
   (junction (at 92.71 55.88) (diameter 0) (color 0 0 0 0)
   )
@@
     (stroke (width 0) (type default))
   )
+  (wire (pts (xy 67.31 55.88) (xy 92.71 55.88))
+    (stroke (width 0) (type default))
+  )
   (wire (pts (xy 82.55 52.07) (xy 102.87 52.07))
     (stroke (width 0) (type default))
   )
-  (wire (pts (xy 96.52 29.21) (xy 96.52 26.67))
+  (wire (pts (xy 76.2 41.91) (xy 102.87 41.91))
+    (stroke (width 0) (type default))
+  )
+  (wire (pts (xy 76.2 41.91) (xy 76.2 68.58))
     (stroke (width 0) (type default))
   )
@@
     (stroke (width 0) (type default))
   )
-  (wire (pts (xy 71.12 41.91) (xy 96.52 41.91))
+  (wire (pts (xy 67.31 76.2) (xy 67.31 91.44))
+    (stroke (width 0) (type default))
+  )
+  (wire (pts (xy 71.12 41.91) (xy 76.2 41.91))
     (stroke (width 0) (type default))
   )
@@
     (stroke (width 0) (type default))
   )
-  (wire (pts (xy 59.69 55.88) (xy 92.71 55.88))
+  (wire (pts (xy 76.2 91.44) (xy 82.55 91.44))
     (stroke (width 0) (type default))
   )
@@
     (stroke (width 0) (type default))
   )
-  (wire (pts (xy 96.52 41.91) (xy 102.87 41.91))
+  (wire (pts (xy 76.2 76.2) (xy 76.2 91.44))
+    (stroke (width 0) (type default))
+  )
+  (wire (pts (xy 67.31 55.88) (xy 67.31 68.58))
+    (stroke (width 0) (type default))
+  )
+  (wire (pts (xy 67.31 91.44) (xy 76.2 91.44))
     (stroke (width 0) (type default))
   )
@@
     (stroke (width 0) (type default))
   )
-  (wire (pts (xy 96.52 36.83) (xy 96.52 41.91))
+  (wire (pts (xy 59.69 55.88) (xy 67.31 55.88))
     (stroke (width 0) (type default))
   )
@@
     )
   )
+  (symbol (lib_id "Device:C") (at 67.31 72.39 0) (unit 1)
+    (in_bom yes) (on_board yes) (dnp no)
+    (property "Reference" "C4" (at 67.31 69.85 0)
+      (effects (font (size 1.27 1.27)) (justify left))
+    )
+    (property "Value" "100nF" (at 67.31 74.93 0)
+      (effects (font (size 1.27 1.27)) (justify left))
+    )
+    (property "Footprint" "Capacitor_SMD:C_0603_1608Metric" (at 68.2752 76.2 0)
+      (effects (font (size 1.27 1.27)) hide)
+    )
+    (property "Datasheet" "~" (at 67.31 72.39 0)
+      (effects (font (size 1.27 1.27)) hide)
+    )
+    (pin "1")
+    (pin "2")
+    (instances
+      (project "PCB"
+        (path "/fd8c8265-4947-4b90-b980-57cac1b7867b"
+          (reference "C4") (unit 1)
+        )
+        (path "/fd8c8265-4947-4b90-b980-57cac1b7867b/70bf9860-66d0-4197-8a28-c71672051aa3"
+          (reference "C9") (unit 1)
+        )
+      )
+    )
+  )
   (symbol (lib_id "Device:R") (at 92.71 62.23 0) (unit 1)
     (in_bom yes) (on_board yes) (dnp no) (fields_autoplaced)
@@
     )
   )
-  (symbol (lib_id "power:GND") (at 96.52 26.67 180) (unit 1)
-    (in_bom yes) (on_board yes) (dnp no) (fields_autoplaced)
-    (property "Reference" "#PWR010" (at 96.52 20.32 0)
-      (effects (font (size 1.27 1.27)) hide)
-    )
-    (property "Value" "GND" (at 96.52 21.59 0)
+  (symbol (lib_id "Device:D") (at 67.31 41.91 0) (unit 1)
+    (in_bom yes) (on_board yes) (dnp no) (fields_autoplaced)
+    (property "Reference" "D7" (at 67.31 35.56 0)
       (effects (font (size 1.27 1.27)))
     )
-    (property "Footprint" "" (at 96.52 26.67 0)
-      (effects (font (size 1.27 1.27)) hide)
-    )
-    (property "Datasheet" "" (at 96.52 26.67 0)
-      (effects (font (size 1.27 1.27)) hide)
-    )
-    (pin "1")
-    (instances
-      (project "PCB"
-        (path "/fd8c8265-4947-4b90-b980-57cac1b7867b"
-          (reference "#PWR010") (unit 1)
-        )
-        (path "/fd8c8265-4947-4b90-b980-57cac1b7867b/70bf9860-66d0-4197-8a28-c71672051aa3"
-          (reference "#PWR010") (unit 1)
-        )
-      )
-    )
-  )
-  (symbol (lib_id "Device:D") (at 67.31 41.91 0) (unit 1)
-    (in_bom yes) (on_board yes) (dnp no) (fields_autoplaced)
-    (property "Reference" "D7" (at 67.31 36.83 0)
+    (property "Value" "BAS16HT1G" (at 67.31 38.1 0)
       (effects (font (size 1.27 1.27)))
     )
-    (property "Value" "1N4818" (at 67.31 39.37 0)
-      (effects (font (size 1.27 1.27)))
-    )
-    (property "Footprint" "Capacitor_SMD:C_0805_2012Metric" (at 67.31 41.91 0)
+    (property "Footprint" "Diode_SMD:D_SOD-323" (at 67.31 41.91 0)
       (effects (font (size 1.27 1.27)) hide)
     )
@@
       (effects (font (size 1.27 1.27)) (justify left))
     )
-    (property "Footprint" "" (at 95.25 78.74 0)
+    (property "Footprint" "Package_TO_SOT_SMD:SOT-23" (at 95.25 78.74 0)
       (effects (font (size 1.27 1.27)) hide)
     )
@@
     )
   )
-  (symbol (lib_id "Device:C") (at 96.52 33.02 180) (unit 1)
-    (in_bom yes) (on_board yes) (dnp no) (fields_autoplaced)
-    (property "Reference" "C4" (at 92.71 33.655 0)
-      (effects (font (size 1.27 1.27)) (justify left))
-    )
-    (property "Value" "100nF" (at 92.71 31.115 0)
-      (effects (font (size 1.27 1.27)) (justify left))
-    )
-    (property "Footprint" "Capacitor_SMD:C_0805_2012Metric" (at 95.5548 29.21 0)
-      (effects (font (size 1.27 1.27)) hide)
-    )
-    (property "Datasheet" "~" (at 96.52 33.02 0)
+  (symbol (lib_id "Device:C") (at 76.2 72.39 0) (unit 1)
+    (in_bom yes) (on_board yes) (dnp no)
+    (property "Reference" "C4" (at 76.2 69.85 0)
+      (effects (font (size 1.27 1.27)) (justify left))
+    )
+    (property "Value" "100nF" (at 76.2 74.93 0)
+      (effects (font (size 1.27 1.27)) (justify left))
+    )
+    (property "Footprint" "Capacitor_SMD:C_0603_1608Metric" (at 77.1652 76.2 0)
+      (effects (font (size 1.27 1.27)) hide)
+    )
+    (property "Datasheet" "~" (at 76.2 72.39 0)
       (effects (font (size 1.27 1.27)) hide)
     )
@@
       (effects (font (size 1.27 1.27)) (justify right))
     )
-    (property "Footprint" "LED_SMD:LED-APA102-2020" (at 92.71 71.12 0)
-      (effects (font (size 1.27 1.27)) hide)
-    )
+    (property "Footprint" "LED_SMD:LED_0805_2012Metric" (at 92.71 71.12 0)
+      (effects (font (size 1.27 1.27)) hide)
+    )

Commit message: Update schematic
Parts:
- C4: footprint Capacitor_SMD:C_0603_1608Metric -> Capacitor_SMD:C_0402_1005Metric
Changed lines of the file:
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@@
       (effects (font (size 1.27 1.27)) (justify left))
     )
-    (property "Footprint" "Capacitor_SMD:C_0603_1608Metric" (at 68.2752 76.2 0)
+    (property "Footprint" "Capacitor_SMD:C_0402_1005Metric" (at 68.2752 76.2 0)
       (effects (font (size 1.27 1.27)) hide)
     )
@@
       (effects (font (size 1.27 1.27)) (justify left))
     )
-    (property "Footprint" "Capacitor_SMD:C_0603_1608Metric" (at 77.1652 76.2 0)
+    (property "Footprint" "Capacitor_SMD:C_0402_1005Metric" (at 77.1652 76.2 0)
       (effects (font (size 1.27 1.27)) hide)
     )

Commit message: Update of PCB and schematic
Parts:
- added J1: 53048-0510, Connector_Molex:Molex_PicoBlade_53048-0510_1x05_P1.25mm_Horizontal, symbol Connector:Conn_01x05_Pin
- C4: footprint Capacitor_SMD:C_0402_1005Metric -> Capacitor_SMD:C_0603_1608Metric
- Q1: value NMOS -> DMN33D8LT-7
Connections:
- net GND: now also J1.5 (Pin_5)
- net +5V_IN renamed +5V_OUT
- net +5V_OUT: now also J1.4 (Pin_4)
- net NRST_IN: no longer names the net of D7.1 (K)
- net NRST_IN: now also J1.1 (Pin_1)
- net SWD_IN renamed SWD_OUT
- net SWD_OUT: now also J1.3 (Pin_3)
- new net SWC_OUT: J1.2 (Pin_2)
Changed lines of the file:
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@@
   (junction (at 76.2 41.91) (diameter 0) (color 0 0 0 0)
   )
-  (junction (at 82.55 52.07) (diameter 0) (color 0 0 0 0)
+  (junction (at 82.55 46.99) (diameter 0) (color 0 0 0 0)
   )
   (junction (at 92.71 91.44) (diameter 0) (color 0 0 0 0)
   )
-  (junction (at 67.31 55.88) (diameter 0) (color 0 0 0 0)
-  )
-  (junction (at 92.71 55.88) (diameter 0) (color 0 0 0 0)
+  (junction (at 67.31 49.53) (diameter 0) (color 0 0 0 0)
+  )
+  (junction (at 92.71 49.53) (diameter 0) (color 0 0 0 0)
   )
   (wire (pts (xy 82.55 82.55) (xy 82.55 81.28))
     (stroke (width 0) (type default))
   )
-  (wire (pts (xy 67.31 55.88) (xy 92.71 55.88))
-    (stroke (width 0) (type default))
-  )
-  (wire (pts (xy 82.55 52.07) (xy 102.87 52.07))
+  (wire (pts (xy 67.31 49.53) (xy 92.71 49.53))
+    (stroke (width 0) (type default))
+  )
+  (wire (pts (xy 82.55 46.99) (xy 102.87 46.99))
     (stroke (width 0) (type default))
   )
@@
     (stroke (width 0) (type default))
   )
+  (wire (pts (xy 92.71 49.53) (xy 102.87 49.53))
+    (stroke (width 0) (type default))
+  )
+  (wire (pts (xy 67.31 76.2) (xy 67.31 91.44))
+    (stroke (width 0) (type default))
+  )
+  (wire (pts (xy 63.5 52.07) (xy 63.5 55.88))
+    (stroke (width 0) (type default))
+  )
+  (wire (pts (xy 71.12 41.91) (xy 76.2 41.91))
+    (stroke (width 0) (type default))
+  )
+  (wire (pts (xy 59.69 52.07) (xy 63.5 52.07))
+    (stroke (width 0) (type default))
+  )
+  (wire (pts (xy 92.71 74.93) (xy 92.71 76.2))
+    (stroke (width 0) (type default))
+  )
+  (wire (pts (xy 76.2 91.44) (xy 82.55 91.44))
+    (stroke (width 0) (type default))
+  )
+  (wire (pts (xy 92.71 86.36) (xy 92.71 91.44))
+    (stroke (width 0) (type default))
+  )
+  (wire (pts (xy 82.55 91.44) (xy 92.71 91.44))
+    (stroke (width 0) (type default))
+  )
+  (wire (pts (xy 82.55 90.17) (xy 82.55 91.44))
+    (stroke (width 0) (type default))
+  )
+  (wire (pts (xy 82.55 81.28) (xy 85.09 81.28))
+    (stroke (width 0) (type default))
+  )
+  (wire (pts (xy 76.2 76.2) (xy 76.2 91.44))
+    (stroke (width 0) (type default))
+  )
+  (wire (pts (xy 67.31 91.44) (xy 76.2 91.44))
+    (stroke (width 0) (type default))
+  )
   (wire (pts (xy 76.2 41.91) (xy 76.2 68.58))
     (stroke (width 0) (type default))
   )
-  (wire (pts (xy 92.71 55.88) (xy 102.87 55.88))
-    (stroke (width 0) (type default))
-  )
-  (wire (pts (xy 67.31 76.2) (xy 67.31 91.44))
-    (stroke (width 0) (type default))
-  )
-  (wire (pts (xy 71.12 41.91) (xy 76.2 41.91))
-    (stroke (width 0) (type default))
-  )
-  (wire (pts (xy 92.71 74.93) (xy 92.71 76.2))
-    (stroke (width 0) (type default))
-  )
-  (wire (pts (xy 76.2 91.44) (xy 82.55 91.44))
-    (stroke (width 0) (type default))
-  )
-  (wire (pts (xy 92.71 86.36) (xy 92.71 91.44))
-    (stroke (width 0) (type default))
-  )
-  (wire (pts (xy 82.55 91.44) (xy 92.71 91.44))
-    (stroke (width 0) (type default))
-  )
-  (wire (pts (xy 82.55 90.17) (xy 82.55 91.44))
-    (stroke (width 0) (type default))
-  )
-  (wire (pts (xy 82.55 81.28) (xy 85.09 81.28))
-    (stroke (width 0) (type default))
-  )
-  (wire (pts (xy 76.2 76.2) (xy 76.2 91.44))
-    (stroke (width 0) (type default))
-  )
-  (wire (pts (xy 67.31 55.88) (xy 67.31 68.58))
-    (stroke (width 0) (type default))
-  )
-  (wire (pts (xy 67.31 91.44) (xy 76.2 91.44))
-    (stroke (width 0) (type default))
-  )
   (wire (pts (xy 59.69 41.91) (xy 63.5 41.91))
     (stroke (width 0) (type default))
   )
-  (wire (pts (xy 59.69 52.07) (xy 82.55 52.07))
-    (stroke (width 0) (type default))
-  )
-  (wire (pts (xy 59.69 55.88) (xy 67.31 55.88))
+  (wire (pts (xy 92.71 49.53) (xy 92.71 58.42))
+    (stroke (width 0) (type default))
+  )
+  (wire (pts (xy 59.69 46.99) (xy 82.55 46.99))
+    (stroke (width 0) (type default))
+  )
+  (wire (pts (xy 82.55 46.99) (xy 82.55 81.28))
+    (stroke (width 0) (type default))
+  )
+  (wire (pts (xy 59.69 49.53) (xy 67.31 49.53))
     (stroke (width 0) (type default))
   )
@@
     (stroke (width 0) (type default))
   )
-  (wire (pts (xy 92.71 55.88) (xy 92.71 58.42))
-    (stroke (width 0) (type default))
-  )
-  (wire (pts (xy 82.55 52.07) (xy 82.55 81.28))
-    (stroke (width 0) (type default))
-  )
-  (wire (pts (xy 59.69 48.26) (xy 102.87 48.26))
+  (wire (pts (xy 67.31 49.53) (xy 67.31 68.58))
+    (stroke (width 0) (type default))
+  )
+  (wire (pts (xy 59.69 44.45) (xy 102.87 44.45))
     (stroke (width 0) (type default))
   )
@@
     (stroke (width 0) (type default))
   )
-  (hierarchical_label "SWD_OUT" (shape output) (at 102.87 52.07 0) (fields_autoplaced)
+  (hierarchical_label "GND" (shape passive) (at 63.5 55.88 270) (fields_autoplaced)
+    (effects (font (size 1.27 1.27)) (justify right))
+  )
+  (hierarchical_label "SWD_OUT" (shape output) (at 102.87 46.99 0) (fields_autoplaced)
     (effects (font (size 1.27 1.27)) (justify left))
   )
-  (hierarchical_label "NRST_IN" (shape input) (at 59.69 41.91 180) (fields_autoplaced)
-    (effects (font (size 1.27 1.27)) (justify right))
-  )
-  (hierarchical_label "SWC_IN" (shape input) (at 59.69 48.26 180) (fields_autoplaced)
-    (effects (font (size 1.27 1.27)) (justify right))
-  )
-  (hierarchical_label "+5V_IN" (shape input) (at 59.69 55.88 180) (fields_autoplaced)
-    (effects (font (size 1.27 1.27)) (justify right))
-  )
-  (hierarchical_label "SWD_IN" (shape input) (at 59.69 52.07 180) (fields_autoplaced)
-    (effects (font (size 1.27 1.27)) (justify right))
-  )
-  (hierarchical_label "+5V_OUT" (shape output) (at 102.87 55.88 0) (fields_autoplaced)
+  (hierarchical_label "+5V_OUT" (shape input) (at 102.87 49.53 0) (fields_autoplaced)
     (effects (font (size 1.27 1.27)) (justify left))
   )
-  (hierarchical_label "SWC_OUT" (shape output) (at 102.87 48.26 0) (fields_autoplaced)
+  (hierarchical_label "SWC_OUT" (shape output) (at 102.87 44.45 0) (fields_autoplaced)
     (effects (font (size 1.27 1.27)) (justify left))
   )
@@
     (effects (font (size 1.27 1.27)) (justify left))
   )
-  (hierarchical_label "GND" (shape output) (at 92.71 93.98 270) (fields_autoplaced)
+  (hierarchical_label "GND" (shape passive) (at 92.71 93.98 270) (fields_autoplaced)
     (effects (font (size 1.27 1.27)) (justify right))
   )
@@
       (effects (font (size 1.27 1.27)) (justify left))
     )
-    (property "Footprint" "Capacitor_SMD:C_0402_1005Metric" (at 68.2752 76.2 0)
+    (property "Footprint" "Capacitor_SMD:C_0603_1608Metric" (at 68.2752 76.2 0)
       (effects (font (size 1.27 1.27)) hide)
     )
@@
       (effects (font (size 1.27 1.27)) (justify left))
     )
-    (property "Value" "NMOS" (at 96.52 83.185 0)
+    (property "Value" "DMN33D8LT-7" (at 96.52 83.185 0)
       (effects (font (size 1.27 1.27)) (justify left))
     )
@@
       (effects (font (size 1.27 1.27)) (justify left))
     )
-    (property "Footprint" "Capacitor_SMD:C_0402_1005Metric" (at 77.1652 76.2 0)
+    (property "Footprint" "Capacitor_SMD:C_0603_1608Metric" (at 77.1652 76.2 0)
       (effects (font (size 1.27 1.27)) hide)
     )
@@
         )
       )
+    )
+  )
+  (symbol (lib_id "Connector:Conn_01x05_Pin") (at 54.61 46.99 0) (unit 1)
+    (in_bom yes) (on_board yes) (dnp no)
+    (property "Reference" "J1" (at 55.245 38.1 0)
+      (effects (font (size 1.27 1.27)))
+    )
+    (property "Value" "53048-0510" (at 54.61 54.61 0)
+      (effects (font (size 1.27 1.27)))
+    )
+    (property "Footprint" "Connector_Molex:Molex_PicoBlade_53048-0510_1x05_P1.25mm_Horizontal" (at 54.61 46.99 0)
+      (effects (font (size 1.27 1.27)) hide)
+    )
+    (property "Datasheet" "~" (at 54.61 46.99 0)
+      (effects (font (size 1.27 1.27)) hide)
+    )
+    (pin "1")
+    (pin "2")
+    (pin "3")
+    (pin "4")
+    (pin "5")
+    (instances
+      (project "PCB"
+        (path "/fd8c8265-4947-4b90-b980-57cac1b7867b"
+          (reference "J1") (unit 1)
+        )
+        (path "/fd8c8265-4947-4b90-b980-57cac1b7867b/70bf9860-66d0-4197-8a28-c71672051aa3"
+          (reference "J4") (unit 1)
+        )
+      )

Commit message: update of directory
Parts:
- added J5: Pin_Header, Connector_PinHeader_2.54mm:PinHeader_1x05_P2.54mm_Horizontal, symbol Connector:Conn_01x05_Pin
- Q1: footprint Package_TO_SOT_SMD:SOT-23 -> Package_TO_SOT_SMD:SOT-523
- renumbered C4 to C9, D7 to D4, J1 to J4
Connections:
- net +5V_OUT: now also J5.4 (Pin_4)
- net GND: now also J5.5 (Pin_5)
- net SWC_OUT: now also J5.2 (Pin_2)
- net SWD_OUT: now also J5.3 (Pin_3)
- net at D4.1 (K), J4.1 (Pin_1): now also J5.1 (Pin_1)
Other:
- moved on the sheet: J4

Commit message: save
Parts:
- renumbered C9 to C12, C4 to C9, D4 to D6, J5 to J1, J4 to J2, Q1 to Q2, R3 to R12, R4 to R16
Changed lines of the file:
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@@
 		(dnp no)
 		(fields_autoplaced yes)
-		(property "Reference" "R4"
+		(property "Reference" "R16"
 			(at 85.09 85.725 0)
 			(effects
@@
 			(project "PCB"
 				(path "/fd8c8265-4947-4b90-b980-57cac1b7867b/70bf9860-66d0-4197-8a28-c71672051aa3"
-					(reference "R4")
+					(reference "R16")
 					(unit 1)
 				)
@@
 		(on_board yes)
 		(dnp no)
-		(property "Reference" "J5"
+		(property "Reference" "J1"
 			(at 36.195 19.05 0)
 			(effects
@@
 			(project "PCB"
 				(path "/fd8c8265-4947-4b90-b980-57cac1b7867b/70bf9860-66d0-4197-8a28-c71672051aa3"
-					(reference "J5")
+					(reference "J1")
 					(unit 1)
 				)
@@
 		(on_board yes)
 		(dnp no)
-		(property "Reference" "C9"
+		(property "Reference" "C12"
 			(at 67.31 69.85 0)
 			(effects
@@
 			(project "PCB"
 				(path "/fd8c8265-4947-4b90-b980-57cac1b7867b/70bf9860-66d0-4197-8a28-c71672051aa3"
-					(reference "C9")
+					(reference "C12")
 					(unit 1)
 				)
@@
 		(dnp no)
 		(fields_autoplaced yes)
-		(property "Reference" "R3"
+		(property "Reference" "R12"
 			(at 95.25 61.595 0)
 			(effects
@@
 			(project "PCB"
 				(path "/fd8c8265-4947-4b90-b980-57cac1b7867b/70bf9860-66d0-4197-8a28-c71672051aa3"
-					(reference "R3")
+					(reference "R12")
 					(unit 1)
 				)
@@
 		(dnp no)
 		(fields_autoplaced yes)
-		(property "Reference" "D4"
+		(property "Reference" "D6"
 			(at 67.31 35.56 0)
 			(effects
@@
 			(project "PCB"
 				(path "/fd8c8265-4947-4b90-b980-57cac1b7867b/70bf9860-66d0-4197-8a28-c71672051aa3"
-					(reference "D4")
+					(reference "D6")
 					(unit 1)
 				)
@@
 		(dnp no)
 		(fields_autoplaced yes)
-		(property "Reference" "Q1"
+		(property "Reference" "Q2"
 			(at 96.52 80.01 0)
 			(effects
@@
 			(project "PCB"
 				(path "/fd8c8265-4947-4b90-b980-57cac1b7867b/70bf9860-66d0-4197-8a28-c71672051aa3"
-					(reference "Q1")
+					(reference "Q2")
 					(unit 1)
 				)
@@
 		(on_board yes)
 		(dnp no)
-		(property "Reference" "C4"
+		(property "Reference" "C9"
 			(at 76.2 69.85 0)
 			(effects
@@
 			(project "PCB"
 				(path "/fd8c8265-4947-4b90-b980-57cac1b7867b/70bf9860-66d0-4197-8a28-c71672051aa3"
-					(reference "C4")
+					(reference "C9")
 					(unit 1)
 				)
@@
 		(on_board yes)
 		(dnp no)
-		(property "Reference" "J4"
+		(property "Reference" "J2"
 			(at 36.195 38.1 0)
 			(effects
@@
 			(project "PCB"
 				(path "/fd8c8265-4947-4b90-b980-57cac1b7867b/70bf9860-66d0-4197-8a28-c71672051aa3"
-					(reference "J4")
-					(unit 1)
-				)
+					(reference "J2")
+					(unit 1)
+				)
