File: Hardware/PCB/Modules/Supply.kicad_sch (KiCad schematic)
At the start: 7 parts, among them U2 LP2985-3.3

Commit message: Update of schematic and PCB
Parts:
- D3: footprint LED_SMD:LED-APA102-2020 -> LED_SMD:LED_0805_2012Metric
- R2: footprint Resistor_SMD:R_0805_2012Metric -> Resistor_SMD:R_0603_1608Metric
Changed lines of the file:
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@@
       (effects (font (size 1.27 1.27)) (justify right))
     )
-    (property "Footprint" "LED_SMD:LED-APA102-2020" (at 142.24 57.15 0)
+    (property "Footprint" "LED_SMD:LED_0805_2012Metric" (at 142.24 57.15 0)
       (effects (font (size 1.27 1.27)) hide)
     )
@@
       (effects (font (size 1.27 1.27)) (justify right))
     )
-    (property "Footprint" "Resistor_SMD:R_0805_2012Metric" (at 144.018 66.04 90)
+    (property "Footprint" "Resistor_SMD:R_0603_1608Metric" (at 144.018 66.04 90)
       (effects (font (size 1.27 1.27)) hide)
     )

Commit message: Update schematic
Parts:
- added C1: 2.2uF, Capacitor_SMD:C_0805_2012Metric, symbol Device:C
- added C2: 10nF, Capacitor_SMD:C_0603_1608Metric, symbol Device:C
- added C3: 4.7uF, Capacitor_SMD:C_0805_2012Metric, symbol Device:C
- added U6: TC1015-1.8VCT713, Package_TO_SOT_SMD:SOT-23-5, symbol Regulator_Linear:TC1015-xCT
Connections:
- net GND: now also C1.2, C2.2, C3.2, U6.2 (GND)
- net at C1.1, R1.2, U2.1 (VIN)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: now also C1.1, U6.1 (VIN), U6.3 (~{SHDN})
- new net: C2.1, U6.4 (Bypass)
- new net +1.8V: C3.1, U6.5 (VOUT)
Other:
- moved on the sheet: C1, C2, C3, D3, R1, R2, U2

Commit message: Update of PCB and schematic
Parts:
- removed C1: 2.2uF, Capacitor_SMD:C_0805_2012Metric, symbol Device:C
- removed C2: 10nF, Capacitor_SMD:C_0603_1608Metric, symbol Device:C
- removed C3: 4.7uF, Capacitor_SMD:C_0805_2012Metric, symbol Device:C
- removed U6: TC1015-1.8VCT713, Package_TO_SOT_SMD:SOT-23-5, symbol Regulator_Linear:TC1015-xCT
Connections:
- net Vin renamed +5V

Commit message: update of directory
Parts:
- C1: value 2.2uF -> 4.7uF; footprint Capacitor_SMD:C_0805_2012Metric -> Capacitor_SMD:C_0603_1608Metric
- C2: value 10nF -> 100nF
- C3: footprint Capacitor_SMD:C_0805_2012Metric -> Capacitor_SMD:C_0603_1608Metric

Commit message: save
Parts:
- removed R1: 18, Resistor_SMD:R_0805_2012Metric, symbol Device:R
- added C18: 4.7uF, Capacitor_SMD:C_0603_1608Metric, symbol Device:C
- added R5: 270, Resistor_SMD:R_0603_1608Metric, symbol Device:R
- added U10: ACS712xLCTR-05B, Package_SO:SOIC-8_3.9x4.9mm_P1.27mm, symbol Sensor_Current:ACS712xLCTR-05B
- renumbered C2 to C4, C1 to C5, C3 to C6, D3 to D2, R2 to R3, U2 to U1
Connections:
- net +5V: now also U10.3 (IP-), U10.4 (IP-)
- net GND: now also C18.2, U10.5 (GND)
- net at C5.1, U1.1 (VIN), U1.3 (ON/~{OFF}): now also U10.1 (IP+), U10.2 (IP+), U10.8 (VCC)
- new net: C18.1, R5.1, U10.7 (VIOUT)
- new net V_{CURRENT}: R5.2
