File: Hardware/PCB/Modules/Temperature.kicad_sch (KiCad schematic)
At the start: 2 parts, among them U4 MCP98243

Commit message: Update schematic
Parts:
- C?: renamed from C2; footprint Capacitor_SMD:C_0603_1608Metric -> Capacitor_SMD:C_0402_1005Metric
- renumbered U4 to U?
Connections:
- net GND_IMU is gone; now on net GND: C?.2
- net GND_TMP is gone; now on net GND: U?.4 (GND), U?.9 (EP/GND)
- net GND: now reaches U?.5 (A2)
- net GND: now also U?.6 (A1), U?.7 (A0)
- net TMP_SCL renamed SCL
- net TMP_SDA renamed SDA
Other:
- note added: "Sensor address : 0x EEPROM address : 0x EEPROM Write protect : 0x"
Changed lines of the file:
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@@
   (junction (at 156.21 66.04) (diameter 0) (color 0 0 0 0)
+  )
+  (junction (at 133.35 100.33) (diameter 0) (color 0 0 0 0)
+  )
+  (junction (at 133.35 97.79) (diameter 0) (color 0 0 0 0)
   )
   (junction (at 151.13 66.04) (diameter 0) (color 0 0 0 0)
   )
   (no_connect (at 161.29 92.71))
-  (wire (pts (xy 134.62 87.63) (xy 140.97 87.63))
+  (bus_entry (at 128.27 83.82) (size -2.54 -2.54)
+    (stroke (width 0) (type default))
+  )
+  (bus_entry (at 125.73 83.82) (size -2.54 -2.54)
+    (stroke (width 0) (type default))
+  )
+  (wire (pts (xy 140.97 100.33) (xy 133.35 100.33))
     (stroke (width 0) (type default))
   )
@@
     (stroke (width 0) (type default))
   )
-  (wire (pts (xy 139.7 78.74) (xy 139.7 81.28))
+  (wire (pts (xy 133.35 100.33) (xy 133.35 102.87))
     (stroke (width 0) (type default))
   )
-  (wire (pts (xy 134.62 85.09) (xy 140.97 85.09))
+  (wire (pts (xy 133.35 97.79) (xy 133.35 100.33))
     (stroke (width 0) (type default))
   )
@@
     (stroke (width 0) (type default))
   )
+  (wire (pts (xy 125.73 87.63) (xy 140.97 87.63))
+    (stroke (width 0) (type default))
+  )
+  (wire (pts (xy 128.27 85.09) (xy 140.97 85.09))
+    (stroke (width 0) (type default))
+  )
   (wire (pts (xy 160.02 60.96) (xy 156.21 60.96))
     (stroke (width 0) (type default))
   )
   (wire (pts (xy 151.13 66.04) (xy 151.13 80.01))
+    (stroke (width 0) (type default))
+  )
+  (wire (pts (xy 140.97 95.25) (xy 133.35 95.25))
+    (stroke (width 0) (type default))
+  )
+  (wire (pts (xy 133.35 95.25) (xy 133.35 97.79))
     (stroke (width 0) (type default))
   )
@@
     (stroke (width 0) (type default))
   )
+  (bus (pts (xy 125.73 81.28) (xy 123.19 81.28))
+    (stroke (width 0) (type default))
+  )
   (wire (pts (xy 153.67 105.41) (xy 153.67 113.03))
+    (stroke (width 0) (type default))
+  )
+  (wire (pts (xy 125.73 83.82) (xy 125.73 87.63))
+    (stroke (width 0) (type default))
+  )
+  (wire (pts (xy 128.27 83.82) (xy 128.27 85.09))
     (stroke (width 0) (type default))
   )
@@
     (stroke (width 0) (type default))
   )
-  (label "GND_IMU" (at 139.7 81.28 0) (fields_autoplaced)
+  (wire (pts (xy 140.97 97.79) (xy 133.35 97.79))
+    (stroke (width 0) (type default))
+  )
+  (bus (pts (xy 123.19 81.28) (xy 115.57 81.28))
+    (stroke (width 0) (type default))
+  )
+  (text "Sensor address : 0x\nEEPROM address : 0x\nEEPROM Write protect : 0x"
+    (at 102.87 100.33 0)
     (effects (font (size 1.27 1.27)) (justify left bottom))
   )
-  (hierarchical_label "GND_TMP" (shape output) (at 152.4 124.46 270) (fields_autoplaced)
+  (label "SCL" (at 134.62 87.63 0) (fields_autoplaced)
+    (effects (font (size 1.27 1.27)) (justify left bottom))
+  )
+  (label "SDA" (at 134.62 85.09 0) (fields_autoplaced)
+    (effects (font (size 1.27 1.27)) (justify left bottom))
+  )
+  (hierarchical_label "{SDA SCL}" (shape bidirectional) (at 115.57 81.28 180) (fields_autoplaced)
+    (effects (font (size 1.27 1.27)) (justify right))
+  )
+  (hierarchical_label "GND" (shape output) (at 152.4 124.46 270) (fields_autoplaced)
     (effects (font (size 1.27 1.27)) (justify right))
   )
@@
     (effects (font (size 1.27 1.27)) (justify left))
   )
-  (hierarchical_label "TMP_SCL" (shape input) (at 134.62 87.63 180) (fields_autoplaced)
+  (hierarchical_label "GND" (shape output) (at 139.7 78.74 270) (fields_autoplaced)
     (effects (font (size 1.27 1.27)) (justify right))
   )
-  (hierarchical_label "TMP_SDA" (shape bidirectional) (at 134.62 85.09 180) (fields_autoplaced)
+  (hierarchical_label "GND" (shape output) (at 133.35 102.87 270) (fields_autoplaced)
     (effects (font (size 1.27 1.27)) (justify right))
   )
   (symbol (lib_id "Device:C") (at 139.7 74.93 0) (unit 1)
     (in_bom yes) (on_board yes) (dnp no) (fields_autoplaced)
-    (property "Reference" "C2" (at 143.51 73.66 0)
+    (property "Reference" "C?" (at 143.51 73.66 0)
       (effects (font (size 1.27 1.27)) (justify left))
     )
@@
       (effects (font (size 1.27 1.27)) (justify left))
     )
-    (property "Footprint" "Capacitor_SMD:C_0603_1608Metric" (at 140.6652 78.74 0)
+    (property "Footprint" "Capacitor_SMD:C_0402_1005Metric" (at 140.6652 78.74 0)
       (effects (font (size 1.27 1.27)) hide)
     )
@@
       (project "PCB"
         (path "/fd8c8265-4947-4b90-b980-57cac1b7867b"
-          (reference "C2") (unit 1)
+          (reference "C?") (unit 1)
         )
         (path "/fd8c8265-4947-4b90-b980-57cac1b7867b/4abdfb61-3b64-4fd4-923e-3cc754423ef0"
@@
         (path "/fd8c8265-4947-4b90-b980-57cac1b7867b/ac97498d-2051-444b-8e34-d771fa4cf1f1"
           (reference "C10") (unit 1)
+        )
+        (path "/fd8c8265-4947-4b90-b980-57cac1b7867b/fd9ec7b9-711c-46f0-80ac-a30badd88661"
+          (reference "C17") (unit 1)
         )
         (path "/fd8c8265-4947-4b90-b980-57cac1b7867b/21016d7c-fd8b-4404-8ef7-6ca90f156ddd"
@@
   (symbol (lib_id "Sensor_Temperature:MCP9808_DFN") (at 151.13 92.71 0) (unit 1)
     (in_bom yes) (on_board yes) (dnp no)
-    (property "Reference" "U4" (at 166.37 89.0621 0)
+    (property "Reference" "U?" (at 166.37 89.0621 0)
       (effects (font (size 1.27 1.27)))
     )
@@
       (project "PCB"
         (path "/fd8c8265-4947-4b90-b980-57cac1b7867b"
+          (reference "U?") (unit 1)
+        )
+        (path "/fd8c8265-4947-4b90-b980-57cac1b7867b/ac97498d-2051-444b-8e34-d771fa4cf1f1"
+          (reference "U6") (unit 1)
+        )
+        (path "/fd8c8265-4947-4b90-b980-57cac1b7867b/fd9ec7b9-711c-46f0-80ac-a30badd88661"
           (reference "U4") (unit 1)
         )
@@
           (reference "U1") (unit 1)
         )
-        (path "/fd8c8265-4947-4b90-b980-57cac1b7867b/ac97498d-2051-444b-8e34-d771fa4cf1f1"
-          (reference "U6") (unit 1)
-        )
       )

Commit message: Update of PCB and schematic
Parts:
- C?: footprint Capacitor_SMD:C_0402_1005Metric -> Capacitor_SMD:C_0603_1608Metric
Connections:
- net VCC_IN renamed +3.3V
Changed lines of the file:
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@@
   (junction (at 152.4 113.03) (diameter 0) (color 0 0 0 0)
-  )
-  (junction (at 156.21 66.04) (diameter 0) (color 0 0 0 0)
   )
   (junction (at 133.35 100.33) (diameter 0) (color 0 0 0 0)
@@
     (stroke (width 0) (type default))
   )
-  (wire (pts (xy 160.02 66.04) (xy 156.21 66.04))
-    (stroke (width 0) (type default))
-  )
   (wire (pts (xy 151.13 113.03) (xy 152.4 113.03))
     (stroke (width 0) (type default))
@@
     (stroke (width 0) (type default))
   )
-  (wire (pts (xy 160.02 60.96) (xy 156.21 60.96))
-    (stroke (width 0) (type default))
-  )
   (wire (pts (xy 151.13 66.04) (xy 151.13 80.01))
     (stroke (width 0) (type default))
@@
     (stroke (width 0) (type default))
   )
-  (wire (pts (xy 156.21 60.96) (xy 156.21 66.04))
-    (stroke (width 0) (type default))
-  )
   (wire (pts (xy 152.4 113.03) (xy 152.4 124.46))
     (stroke (width 0) (type default))
   )
-  (wire (pts (xy 156.21 66.04) (xy 151.13 66.04))
+  (wire (pts (xy 151.13 66.04) (xy 160.02 66.04))
     (stroke (width 0) (type default))
   )
@@
     (effects (font (size 1.27 1.27)) (justify right))
   )
-  (hierarchical_label "GND" (shape output) (at 152.4 124.46 270) (fields_autoplaced)
+  (hierarchical_label "GND" (shape passive) (at 152.4 124.46 270) (fields_autoplaced)
     (effects (font (size 1.27 1.27)) (justify right))
   )
-  (hierarchical_label "VCC_IN" (shape input) (at 160.02 66.04 0) (fields_autoplaced)
+  (hierarchical_label "+3.3V" (shape input) (at 160.02 66.04 0) (fields_autoplaced)
     (effects (font (size 1.27 1.27)) (justify left))
   )
-  (hierarchical_label "VCC_OUT" (shape output) (at 160.02 60.96 0) (fields_autoplaced)
-    (effects (font (size 1.27 1.27)) (justify left))
-  )
-  (hierarchical_label "GND" (shape output) (at 139.7 78.74 270) (fields_autoplaced)
+  (hierarchical_label "GND" (shape passive) (at 139.7 78.74 270) (fields_autoplaced)
     (effects (font (size 1.27 1.27)) (justify right))
   )
-  (hierarchical_label "GND" (shape output) (at 133.35 102.87 270) (fields_autoplaced)
+  (hierarchical_label "GND" (shape passive) (at 133.35 102.87 270) (fields_autoplaced)
     (effects (font (size 1.27 1.27)) (justify right))
   )
@@
       (effects (font (size 1.27 1.27)) (justify left))
     )
-    (property "Footprint" "Capacitor_SMD:C_0402_1005Metric" (at 140.6652 78.74 0)
+    (property "Footprint" "Capacitor_SMD:C_0603_1608Metric" (at 140.6652 78.74 0)
       (effects (font (size 1.27 1.27)) hide)
     )

Commit message: update of directory
Parts:
- gave numbers to parts that had none: 2

Commit message: save
Parts:
- renumbered C11 to C14, U1 to U4
Changed lines of the file:
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@@
 		(dnp no)
 		(fields_autoplaced yes)
-		(property "Reference" "C11"
+		(property "Reference" "C14"
 			(at 143.51 73.66 0)
 			(effects
@@
 			(project "PCB"
 				(path "/fd8c8265-4947-4b90-b980-57cac1b7867b/21016d7c-fd8b-4404-8ef7-6ca90f156ddd"
-					(reference "C11")
+					(reference "C14")
 					(unit 1)
 				)
@@
 		(on_board yes)
 		(dnp no)
-		(property "Reference" "U1"
+		(property "Reference" "U4"
 			(at 166.37 89.0621 0)
 			(effects
@@
 			(project "PCB"
 				(path "/fd8c8265-4947-4b90-b980-57cac1b7867b/21016d7c-fd8b-4404-8ef7-6ca90f156ddd"
-					(reference "U1")
+					(reference "U4")
 					(unit 1)
 				)
