File: Hardware/PCB/PCB.kicad_sch (KiCad schematic)
At the start: 75 parts, among them P1 USB_C_Plug, U1 STM32F423RHTx

Commit message: Add keyboard submodule
Parts:
- removed D1: D, symbol Device:D
- removed D10, D11, D12, D13, D14, D15, D16, D17, D18, D19, D2, D20, D21, D22, D23, D24, D25, D26, D27, D28, D29, D3, D30, D31, D32, D33, D34, D35, D36, D37, D38, D39, D4, D40, D41, D42, D43, D44, D45, D46, D47, D48, D49, D5, D50, D51, D52, D53, D54, D55, D56, D57, D58, D59, D6, D60, D61, D62, D63, D64, D65, D66, D67, D68, D69, D7, D70, D71, D72, D73, D8, D9: SK6812MINI, LED_SMD:LED_SK6812MINI_PLCC4_3.5x3.5mm_P1.75mm, symbol LED:SK6812MINI
- P1: footprint (none) -> Diode_SMD:D_SMA
Other:
- added sheet Key (Key.kicad_sch)

Commit message: first schematic
Parts:
- removed U1: STM32F423RHTx, Package_QFP:LQFP-64_10x10mm_P0.5mm, symbol MCU_ST_STM32F4:STM32F423RHTx
- added C5, C7, C8: 100nF, Capacitor_SMD:C_0805_2012Metric, symbol Device:C
- added C6: 470nF, Capacitor_SMD:C_0805_2012Metric, symbol Device:C
- added J1: Conn_01x05_Pin, Connector_PinHeader_2.54mm:PinHeader_1x05_P2.54mm_Horizontal, symbol Connector:Conn_01x05_Pin
- added U3: STM32F303RETx, Package_QFP:LQFP-64_10x10mm_P0.5mm, symbol MCU_ST_STM32F3:STM32F303RETx
- P1: footprint Diode_SMD:D_SMA -> Connector_USB:USB_C_Plug_JAE_DX07P024AJ1
Connections:
- net GND: now reaches P1.A1 (GND), P1.A12 (GND), P1.B1 (GND), P1.B12 (GND)
- net GND: now also P1.S1 (SHIELD), C5.2, C6.2, C7.2, C8.2, J1.5 (Pin_5), U3.12 (VSSA), U3.18 (VSS), U3.31 (VSS), U3.47 (VSS), U3.63 (VSS)
- net +5V: now reaches P1.A4 (VBUS), P1.A9 (VBUS), P1.B4 (VBUS), P1.B9 (VBUS)
- new net +3.3V: C5.1, C6.1, C7.1, C8.1, U3.1 (VBAT), U3.13 (VDDA), U3.19 (VDD), U3.32 (VDD), U3.48 (VDD), U3.64 (VDD)
- new net Programming/+5V_IN: J1.1 (Pin_1)
- new net Programming/NRST_IN: J1.2 (Pin_2)
- new net Programming/SWC_IN: J1.4 (Pin_4)
- new net Programming/SWD_IN: J1.3 (Pin_3)
Other:
- sheet Key renamed Key_1U
- added sheet Programming (Modules/Programming_sch.kicad_sch)
- added sheet Supply (Modules/Supply.kicad_sch)
- sheet Key_1U: file Key.kicad_sch -> Modules/Key.kicad_sch
- moved on the sheet: P1

Commit message: Update of schematic and PCB
Parts:
- removed C5, C7, C8: 100nF, Capacitor_SMD:C_0805_2012Metric, symbol Device:C
- removed C6: 470nF, Capacitor_SMD:C_0805_2012Metric, symbol Device:C
- removed U3: STM32F303RETx, Package_QFP:LQFP-64_10x10mm_P0.5mm, symbol MCU_ST_STM32F3:STM32F303RETx
- J1: value Conn_01x05_Pin -> 53048-0510; footprint Connector_PinHeader_2.54mm:PinHeader_1x05_P2.54mm_Horizontal -> Connector_Molex:Molex_PicoBlade_53048-0510_1x05_P1.25mm_Horizontal
Other:
- added sheet IMU (IMU.kicad_sch)
- added sheet MCU (MCU.kicad_sch.kicad_sch)
- added sheet Temperature (Temperature.kicad_sch)

Commit message: Update schematic
Connections:
- net +5V renamed Programming/+5V_OUT
Other:
- added sheet Multimeter (Modules/Multimeter.kicad_sch)
- added sheet OLED (Modules/OLED.kicad_sch)
- added sheet UART (Modules/UART.kicad_sch)
- sheet IMU: file IMU.kicad_sch -> Modules/IMU.kicad_sch
- sheet IMU ports: added +1.8V, +3.3V, GND, {SDA SCL}; removed GND_IMU, IMU_SCL, IMU_SDA, VCC_IN, VCC_OUT
- sheet MCU: file MCU.kicad_sch.kicad_sch -> Modules/MCU.kicad_sch.kicad_sch
- sheet MCU ports: added +3.3V, GND, SWC, SWD, {SDA SCL}; removed GND_MCU, SCL_MCU, SDA_MCU, VCC_IN, VCC_OUT
- sheet Supply ports: added +1.8V; removed none
- sheet Temperature: file Temperature.kicad_sch -> Modules/Temperature.kicad_sch
- sheet Temperature ports: added GND, {SDA SCL}; removed GND_TMP, TMP_SCL, TMP_SDA

Commit message: Update of PCB and schematic
Parts:
- removed J1: 53048-0510, Connector_Molex:Molex_PicoBlade_53048-0510_1x05_P1.25mm_Horizontal, symbol Connector:Conn_01x05_Pin
- removed P1: USB_C_Plug, Connector_USB:USB_C_Plug_JAE_DX07P024AJ1, symbol Connector:USB_C_Plug
Other:
- removed sheet UART
- added sheet I2C_LevelShifter1 (LevelShifter.kicad_sch)
- added sheet UART_Slot (UART_Slot.kicad_sch)
- added sheet USB_Slot (USB_Slot.kicad_sch)
- sheet IMU ports: added none; removed +1.8V
- sheet MCU ports: added RX, TX; removed none
- sheet Multimeter ports: added +5V; removed VCC_IN, VCC_OUT
- sheet OLED ports: added +3.3V, +5V; removed VCC_IN, VCC_OUT
- sheet Programming ports: added none; removed +5V_IN, NRST_IN, SWC_IN, SWD_IN
- sheet Supply ports: added +5V; removed +1.8V
- sheet Temperature ports: added +3.3V; removed VCC_IN, VCC_OUT

Commit message: save
Other:
- added sheet EEPROM (Modules/EEPROM.kicad_sch)
- sheet Supply ports: added V_{CURRENT}; removed none
Changed lines of the file:
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@@
+			)
+		)
+		(pin "V_{CURRENT}" output
+			(at 96.52 45.72 0)
+			(effects
+				(font
+					(size 1.27 1.27)
+				)
+				(justify right)
 			)
 		)
@@
 				)
 			)
+		)
+	)
+	(sheet
+		(at 195.58 96.52)
+		(size 12.7 17.78)
+		(fields_autoplaced yes)
+		(stroke
+			(width 0.1524)
+			(type solid)
+		)
+		(fill
+			(color 0 0 0 0.0000)
+		)
+		(property "Sheetname" "EEPROM"
+			(at 194.8684 114.3 90)
+			(effects
+				(font
+					(size 1.27 1.27)
+				)
+				(justify left bottom)
+			)
+		)
+		(property "Sheetfile" "Modules/EEPROM.kicad_sch"
+			(at 208.8646 114.3 90)
+			(effects
+				(font
+					(size 1.27 1.27)
+				)
+				(justify left top)
+				(hide yes)
+			)
+		)
+		(pin "ADC_OUT" output
+			(at 201.93 114.3 270)
+			(effects
+				(font
+					(size 1.27 1.27)
+				)
+				(justify left)
+			)
+		)
+		(pin "GND" output
+			(at 198.12 114.3 270)
+			(effects
+				(font
+					(size 1.27 1.27)
+				)
+				(justify left)
+			)
+		)
+		(pin "+5V" input
+			(at 198.12 96.52 90)
+			(effects
+				(font
+					(size 1.27 1.27)
+				)
+				(justify right)
+			)
+		)
+		(instances
+			(project "PCB"
+				(path "/fd8c8265-4947-4b90-b980-57cac1b7867b"
+					(page "11")
+				)
+			)
