File: Hardware/PCB/UART_Slot.kicad_sch (KiCad schematic)
At the start: 5 parts, among them J3 USB_C_Receptacle_PowerOnly_6P, U5 USBLC6-2P6, U7 FT231XQ

Commit message: update of directory
Parts:
- R17: footprint Resistor_SMD:R_0402_1005Metric -> Resistor_SMD:R_0603_1608Metric
- renumbered J3 to J1, U5 to U6

Commit message: save
Parts:
- removed J1: USB_C_Receptacle_PowerOnly_6P, Connector_USB:USB_C_Receptacle_GCT_USB4125-xx-x_6P_TopMnt_Horizontal, symbol Connector:USB_C_Receptacle_PowerOnly_6P
- added D10, D9: LED, LED_SMD:LED_0805_2012Metric, symbol Device:LED
- added J4: USB_C_Receptacle_USB2.0_16P, Connector_USB:USB_C_Receptacle_GCT_USB4085, symbol Connector:USB_C_Receptacle_USB2.0_16P
- added R35, R36: 270, Resistor_SMD:R_0603_1608Metric, symbol Device:R
- added R37, R38: 22, Resistor_SMD:R_0603_1608Metric, symbol Device:R
- renumbered R17 to R34, U6 to U7, U7 to U8
Connections:
- net GND: now also U7.2 (GND), U8.13 (GND), U8.21 (GND), U8.3 (GND), J4.A1 (GND), J4.A12 (GND), J4.B1 (GND), J4.B12 (GND), J4.S1 (SHIELD)
- net VBus: now also J4.A4 (VBUS), J4.A9 (VBUS), J4.B4 (VBUS), J4.B9 (VBUS); no longer R34.1
- net at U7.1 (I/O1): now also U8.9 (USBDM); no longer U8.8 (USBDP)
- net at U7.3 (I/O2): now also U8.8 (USBDP); no longer U8.9 (USBDM)
- net at U7.4 (I/O2): now also R38.2
- net at U7.6 (I/O1): now also R37.2
- net +3.3V: now reaches U8.10 (3V3OUT)
- net +3.3V: now also R34.1, R35.1, R36.1
- net at U8.14 (CBUS1): now also D9.1 (K)
- net at U8.15 (CBUS0): now also D10.1 (K)
- new net: J4.A7 (D-), J4.B7 (D-), R37.1
- new net: D10.2 (A), R36.2
- new net: D9.2 (A), R35.2
- new net: J4.A6 (D+), J4.B6 (D+), R38.1
- no-connect marks 4 -> 11
Other:
- moved on the sheet: D8
