File: Hardware/PCB/USB_Slot.kicad_sch (KiCad schematic)
At the start: 2 parts, among them J3 USB_C_Receptacle_PowerOnly_6P, U5 USBLC6-2P6

Commit message: save
Parts:
- removed J3: USB_C_Receptacle_PowerOnly_6P, Connector_USB:USB_C_Receptacle_GCT_USB4125-xx-x_6P_TopMnt_Horizontal, symbol Connector:USB_C_Receptacle_PowerOnly_6P
- added D7: D, Diode_SMD:D_0805_2012Metric, symbol Device:D
- added J3: USB_C_Receptacle_USB2.0_16P, Connector_USB:USB_C_Receptacle_GCT_USB4085, symbol Connector:USB_C_Receptacle_USB2.0_16P
- added R39, R40: 22, Resistor_SMD:R_0603_1608Metric, symbol Device:R
- renumbered U5 to U6
Connections:
- net +5V: now also D7.1 (K); no longer U6.5 (VBUS)
- net DATA+: now also U6.3 (I/O2); no longer U6.1 (I/O1)
- net DATA-: now also U6.1 (I/O1); no longer U6.3 (I/O2)
- net GND: now also J3.A1 (GND), J3.A12 (GND), J3.B1 (GND), J3.B12 (GND), J3.S1 (SHIELD)
- net at U6.4 (I/O2): now also R39.2
- net at U6.6 (I/O1): now also R40.2
- new net: J3.A6 (D+), J3.B6 (D+), R39.1
- new net: J3.A7 (D-), J3.B7 (D-), R40.1
- new net VBus: D7.2 (A), J3.A4 (VBUS), J3.A9 (VBUS), J3.B4 (VBUS), J3.B9 (VBUS), U6.5 (VBUS)
- no-connect marks 0 -> 4
