File: Hardware/V1.0_Prototype/PCB.kicad_sch (KiCad schematic)
At the start: 0 parts

Commit message: update repo, add proto PCB
Other:
- removed sheet I2C_LevelShifter1
- added sheet Key_1U1 (Modules/Key.kicad_sch)
- added sheet Key_1U2 (Modules/Key.kicad_sch)
- added sheet Key_1U3 (Modules/Key.kicad_sch)
- added sheet RTC (Modules/RTC.kicad_sch)
- sheet EEPROM ports: added +3.3V, {SPI}; removed +5V, ADC_OUT
- sheet IMU ports: added {I2C}; removed {SDA SCL}
- sheet MCU ports: added {I2C}, {SPI}; removed {SDA SCL}
- sheet OLED ports: added {I2C}; removed {SDA SCL}
- sheet Programming ports: added +3.3V, JTDI, NRST, SWCLK, SWDIO, SWO, VCP_RX, VCP_TX; removed NRST_OUT, SWC_OUT, SWD_OUT
- sheet Supply ports: added +5V_{OUT}; removed Vin
- sheet Temperature ports: added {I2C}; removed {SDA SCL}
- sheet UART_Slot ports: added +5V_USB; removed +5V
- sheet USB_Slot ports: added +5V_USB; removed +5V
