File: Hardware/V1.0_Prototype/Modules/MCU.kicad_sch.kicad_sch (KiCad schematic)
At the start: 18 parts, among them U2 STM32F303RETx, X1 ECS-2520MV-250-DN-TR

Commit message: update repo, add proto PCB
Parts:
- removed C1, C11, C13, C2, C3: 100nF, Capacitor_SMD:C_0603_1608Metric, symbol Device:C
- removed R10, R6: 0, Resistor_SMD:R_0603_1608Metric, symbol Device:R
- removed R11: 4.7k, Resistor_SMD:R_0603_1608Metric, symbol Device:R
- removed R20: 220, Resistor_SMD:R_0603_1608Metric, symbol Device:R
- removed R26: 10, Resistor_SMD:R_0603_1608Metric, symbol Device:R
- added C21, C22, C23, C24, C25: 100nF, Capacitor_SMD:C_0603_1608Metric_Pad1.08x0.95mm_HandSolder, symbol Device:C
- added R16, R17, R18: 0, Resistor_SMD:R_0805_2012Metric_Pad1.20x1.40mm_HandSolder, symbol Device:R
- added R41, R42: 4.7k, Resistor_SMD:R_0805_2012Metric_Pad1.20x1.40mm_HandSolder, symbol Device:R
- C15, C7: footprint Capacitor_SMD:C_0603_1608Metric -> Capacitor_SMD:C_0603_1608Metric_Pad1.08x0.95mm_HandSolder
- R13, R14, R15, R22: footprint Resistor_SMD:R_0603_1608Metric -> Resistor_SMD:R_0805_2012Metric_Pad1.20x1.40mm_HandSolder
Connections:
- net +3.3V: now also C21.1, C22.1, C23.1, C24.1, C25.1
- net GND: now also C21.2, C22.2, C23.2, C24.2, C25.2, R17.1
- net IR_LED: now also R42.2
- net SDA: now also R41.2
- net SWC: now also R16.2
- net USB+: now also R14.2; no longer R13.2
- net USB-: now also R13.2; no longer R14.2
- net VCC_MCU: now also R41.1
- net at U2.49 (PA14): now also R16.1
- net at U2.60 (BOOT0): now also R17.2
- net at U2.5 (PF0): now also R18.2
- net CLK: now reaches U2.51 (PC10)
- net MISO: now reaches U2.52 (PC11)
- net MOSI: now reaches U2.53 (PC12)
- net at U2.62 (PB9): now also R42.1
- net at X1.3 (OUT): now also R18.1
